Commit message: Created base and wheels from scratch

File: urdf/hello_robot.urdf (robot description, URDF)
Before this commit: robot myfirst, 1 links, 0 joints
Links:
- added link left_front_wheel; visual cylinder length=.00325 radius=.00325
- added link left_rear_wheel; visual cylinder length=.00325 radius=.00325
- added link right_front_wheel; visual cylinder length=.00325 radius=.00325
- added link right_rear_wheel; visual cylinder length=.00325 radius=.00325
- link base_link: geometry visual box size=.023 .026 0.005
Joints:
- added joint base_to_left_front_wheel: type fixed, parent base_link, child left_front_wheel
- added joint base_to_left_rear_wheel: type fixed, parent base_link, child left_rear_wheel
- added joint base_to_right_front_wheel: type fixed, parent base_link, child right_front_wheel
- added joint base_to_right_rear_wheel: type fixed, parent base_link, child right_rear_wheel

Commit message: Rviz working, gazebo not working

File: urdf/hello_robot.urdf (robot description, URDF)
Before this commit: robot hello_robot, 5 links, 4 joints
Links:
- link base_link: geometry visual box size=0.23 0.26 0.01
- link left_front_wheel: geometry collision cylinder length=0.0325 radius=0.0325; visual cylinder length=0.0325 radius=0.0325
- link left_rear_wheel: geometry collision cylinder length=0.0325 radius=0.0325; visual cylinder length=0.0325 radius=0.0325
- link right_front_wheel: geometry collision cylinder length=0.0325 radius=0.0325; visual cylinder length=0.0325 radius=0.0325
- link right_rear_wheel: geometry collision cylinder length=0.0325 radius=0.0325; visual cylinder length=0.0325 radius=0.0325
Joints:
- joint left_front_wheel_joint: origin xyz=0.007666666666666666 0.014624999999999999 -0.00325 rpy=0 0 0 -> xyz=0.07666666666666667 0.14625 -0.0325 rpy=0 0 0
- joint left_rear_wheel_joint: origin xyz=-0.007666666666666666 0.014624999999999999 -0.00325 rpy=0 0 0 -> xyz=-0.07666666666666667 0.14625 -0.0325 rpy=0 0 0
- joint right_front_wheel_joint: origin xyz=0.007666666666666666 -0.014624999999999999 -0.00325 rpy=0 0 0 -> xyz=0.07666666666666667 -0.14625 -0.0325 rpy=0 0 0
- joint right_rear_wheel_joint: origin xyz=-0.007666666666666666 -0.014624999999999999 -0.00325 rpy=0 0 0 -> xyz=-0.07666666666666667 -0.14625 -0.0325 rpy=0 0 0

File: urdf/hello_robot.xacro (robot description, xacro)
@@ -1,13 +1,16 @@
 <?xml version="1.0"?>
 <robot name="hello_robot" xmlns:xacro="http://www.ros.org/wiki/xacro">
-  <xacro:property name="baselen" value="0.023" />
-  <xacro:property name="basewidth" value="0.026" />
-  <xacro:property name="basethick" value="0.001" />
-  <xacro:property name="wheeldiam" value="0.0065" />
-  <xacro:property name="wheelwidth" value="0.00325" />
+  <xacro:property name="baselen" value="0.23" />
+  <xacro:property name="basewidth" value="0.26" />
+  <xacro:property name="basethick" value="0.01" />
+  <xacro:property name="wheeldiam" value="0.065" />
+  <xacro:property name="wheelwidth" value="0.0325" />
   <xacro:property name="pi" value="3.1415" />
   <xacro:property name="mass" value="1.45" />
   <material name="white">
     <color rgba="1 1 1 1"/>
+  </material>
+  <material name="black">
+    <color rgba=".05 .05 .05 1"/>
   </material>
   <xacro:macro name="default_inertial" params="mass">

Commit message: xacro hello_robot.xacro > hello_robot.urdf

File: urdf/hello_robot.urdf (robot description, URDF)
Before this commit: robot hello_robot, 5 links, 4 joints
Links:
- removed link left_rear_wheel
- removed link right_rear_wheel
- added link left_back_wheel, mass 0.1; collision cylinder length=0.0325 radius=0.0325; visual cylinder length=0.0325 radius=0.0325
- added link right_back_wheel, mass 0.1; collision cylinder length=0.0325 radius=0.0325; visual cylinder length=0.0325 radius=0.0325
- link base_link: mass None -> 1; geometry collision box size=0.23 0.26 0.01; visual box size=0.23 0.26 0.01
- link left_front_wheel: mass 1 -> 0.1
- link right_front_wheel: mass 1 -> 0.1
Joints:
- removed joint left_rear_wheel_joint
- removed joint right_rear_wheel_joint
- added joint left_back_wheel_joint: type continuous, parent base_link, child left_back_wheel, origin xyz=-0.07666666666666667 0.14625 -0.0325 rpy=0 0 0, axis 0 1 0
- added joint right_back_wheel_joint: type continuous, parent base_link, child right_back_wheel, origin xyz=-0.07666666666666667 -0.14625 -0.0325 rpy=0 0 0, axis 0 1 0
