Commit message: basic xacro file completed

File: urdf/hello_robot.xacro (robot description, xacro)
@@ -3,9 +3,9 @@
   <xacro:property name="baselen" value="0.023" />
   <xacro:property name="basewidth" value="0.026" />
-  <xacro:property name="basethick" value="0.005" />
+  <xacro:property name="basethick" value="0.001" />
   <xacro:property name="wheeldiam" value="0.0065" />
-  <xacro:property name="wheelwidth" value="0.0065" />
+  <xacro:property name="wheelwidth" value="0.00325" />
   <xacro:property name="pi" value="3.1415" />
-  <xacro:property name="mass" value="1" />
+  <xacro:property name="mass" value="1.45" />
   <material name="white">
     <color rgba="1 1 1 1"/>
@@ -25,5 +25,5 @@
     </visual>
   </link>
-  <xacro:macro name="wheel" params="prefix suffix reflect">
+  <xacro:macro name="wheel" params="prefix suffix reflectfrontback reflectside">
     <link name="${prefix}_${suffix}_wheel">
       <visual>
@@ -46,8 +46,10 @@
       <parent link="base_link"/>
       <child link="${prefix}_${suffix}_wheel"/>
-      <origin xyz="${baselen*reflect/3} ${.015} -${wheeldiam/2}" rpy="0 0 0"/>
+      <origin xyz="${baselen*reflectfrontback/3} ${((basewidth/2)+wheelwidth/2)*reflectside} ${-wheeldiam/2}" rpy="0 0 0"/>
     </joint>
   </xacro:macro>
-  <xacro:wheel prefix="left" suffix="front" reflect="1"/>
-  <xacro:wheel prefix="left" suffix="rear" reflect="-1"/>
+  <xacro:wheel prefix="left" suffix="front" reflectfrontback="1" reflectside="1"/>
+  <xacro:wheel prefix="left" suffix="rear" reflectfrontback="-1" reflectside="1"/>
+  <xacro:wheel prefix="right" suffix="front" reflectfrontback="1" reflectside="-1"/>
+  <xacro:wheel prefix="right" suffix="rear" reflectfrontback="-1" reflectside="-1"/>
 </robot>

Commit message: Gazebo working but need to tune driving

File: urdf/hello_robot.xacro (robot description, xacro)
@@ -27,4 +27,10 @@
       <material name="white"/>
     </visual>
+    <collision>
+      <geometry>
+        <box size="${baselen} ${basewidth} ${basethick}" />
+      </geometry>
+    </collision>
+    <xacro:default_inertial mass="10"/>
   </link>
   <xacro:macro name="wheel" params="prefix suffix reflectfrontback reflectside">
@@ -51,8 +57,34 @@
       <origin xyz="${baselen*reflectfrontback/3} ${((basewidth/2)+wheelwidth/2)*reflectside} ${-wheeldiam/2}" rpy="0 0 0"/>
     </joint>
+        <!-- This block provides the simulator (Gazebo) with information on a few additional
+    physical properties. See http://gazebosim.org/tutorials/?tut=ros_urdf for more-->
+    <gazebo reference="${prefix}_${suffix}_wheel">
+      <mu1 value="200.0"/>
+      <mu2 value="100.0"/>
+      <kp value="10000000.0" />
+      <kd value="1.0" />
+      <material>Gazebo/Grey</material>
+    </gazebo>
+    <!-- This block connects the wheel joint to an actuator (motor), which informs both
+    simulation and visualization of the robot -->
+    <transmission name="${prefix}_${suffix}_wheel_trans">
+      <type>transmission_interface/SimpleTransmission</type>
+      <actuator name="${prefix}_${suffix}_wheel_motor">
+        <mechanicalReduction>1</mechanicalReduction>
+      </actuator>
+      <joint name="${prefix}_${suffix}_wheel_joint">
+        <hardwareInterface>VelocityJointInterface</hardwareInterface>
+      </joint>
+    </transmission>
   </xacro:macro>
   <xacro:wheel prefix="left" suffix="front" reflectfrontback="1" reflectside="1"/>
-  <xacro:wheel prefix="left" suffix="rear" reflectfrontback="-1" reflectside="1"/>
+  <xacro:wheel prefix="left" suffix="back" reflectfrontback="-1" reflectside="1"/>
   <xacro:wheel prefix="right" suffix="front" reflectfrontback="1" reflectside="-1"/>
-  <xacro:wheel prefix="right" suffix="rear" reflectfrontback="-1" reflectside="-1"/>
+  <xacro:wheel prefix="right" suffix="back" reflectfrontback="-1" reflectside="-1"/>
+  <!-- Gazebo plugin for ROS Control -->
+  <gazebo>
+    <plugin name="gazebo_ros_control" filename="libgazebo_ros_control.so">
+      <robotNamespace>/</robotNamespace>
+    </plugin>
+  </gazebo>
 </robot>

Commit message: Update of parameters

File: urdf/hello_robot.xacro (robot description, xacro)
@@ -7,5 +7,4 @@
   <xacro:property name="wheelwidth" value="0.0325" />
   <xacro:property name="pi" value="3.1415" />
-  <xacro:property name="mass" value="1.45" />
   <material name="white">
     <color rgba="1 1 1 1"/>
@@ -32,5 +31,5 @@
       </geometry>
     </collision>
-    <xacro:default_inertial mass="10"/>
+    <xacro:default_inertial mass="1"/>
   </link>
   <xacro:macro name="wheel" params="prefix suffix reflectfrontback reflectside">
@@ -49,5 +48,5 @@
         </geometry>
       </collision>
-      <xacro:default_inertial mass="1"/>
+      <xacro:default_inertial mass="0.1"/>
     </link>
     <joint name="${prefix}_${suffix}_wheel_joint" type="continuous">

Commit message: Updated inertias for base and wheels

File: urdf/hello_robot.xacro (robot description, xacro)
@@ -13,8 +13,37 @@
     <color rgba=".05 .05 .05 1"/>
   </material>
-  <xacro:macro name="default_inertial" params="mass">
+  <!-- ======================= Intertial macros ===============================-->
+  <!-- ===================== Cylinder intertia xacro =============================
+  Xacro with the intertial block of a cylinder. For more detail information and usage, see:
+    https://github.com/pxalcantara/mobile_robot_description/wiki/Inertia-xacro
+  params:
+  - m [float]: link mass;
+  - r [float]: cylinder radius;
+  - l [float]: cylinder lenght (height);
+  -->
+  <xacro:macro name="wheel_inertia" params="m r l o_xyz:='0.0 0.0 0.0' o_rpy:='0.0 0.0 0.0'">
     <inertial>
-      <mass value="${mass}" />
-      <inertia ixx="1.0" ixy="0.0" ixz="0.0" iyy="1.0" iyz="0.0" izz="1.0" />
+      <mass value="${m}"/>
+      <inertia ixx="${m*(3*r*r+l*l)/12}" ixy = "0" ixz = "0"
+               iyy="${m*(3*r*r+l*l)/12}" iyz = "0" izz="${m*r*r/2}"/>
+      <origin xyz="${o_xyz}" rpy="${o_rpy}" />
+    </inertial>
+  </xacro:macro>
+  <!-- ===================== Box intertia xacro ==================================
+  Xacro with the intertial block of a box. For more detail information and usage, see:
+    https://github.com/pxalcantara/mobile_robot_description/wiki/Inertia-xacro
+  params:
+  - m [float]: link mass;
+  - x [float]: link dimension on the X-axis;
+  - y [float]: link dimension on the Y-axis;
+  - z [float]: link dimension on the Z-axis;
+-->
+<xacro:macro name="base_inertia" params="m x y z o_xyz:='0.0 0.0 0.0' o_rpy:='0.0 0.0 0.0'">
+    <inertial>
+      <mass value="${m}"/>
+      <inertia ixx="${m / 12.0 * (y*y + z*z)}" ixy="0.0" ixz="0.0"
+               iyy="${m / 12.0 * (x*x + z*z)}" iyz="0.0"
+               izz="${m / 12.0 * (x*x + y*y)}"/>
+      <origin xyz="${o_xyz}" rpy="${o_rpy}" />
     </inertial>
   </xacro:macro>
@@ -31,5 +60,8 @@
       </geometry>
     </collision>
-    <xacro:default_inertial mass="1"/>
+    <xacro:base_inertia m="1"
+    x="${baselen}" y="${basewidth}" z="${basethick}"
+    o_xyz="0.0 0.0 0.0" o_rpy="0.0 0.0 0.0"
+    />
   </link>
   <xacro:macro name="wheel" params="prefix suffix reflectfrontback reflectside">
@@ -48,5 +80,7 @@
         </geometry>
       </collision>
-      <xacro:default_inertial mass="0.1"/>
+      <xacro:wheel_inertia m="0.1" r="${wheeldiam/2}" l="${wheelwidth}"
+      o_xyz="0.0 0.0 0.0" o_rpy="0.0 0.0 0.0"
+      />
     </link>
     <joint name="${prefix}_${suffix}_wheel_joint" type="continuous">

Commit message: Working on urdf and organizing

File: urdf/hello_robot.xacro (robot description, xacro)
@@ -1,51 +1,14 @@
 <?xml version="1.0"?>
 <robot name="hello_robot" xmlns:xacro="http://www.ros.org/wiki/xacro">
-  <xacro:property name="baselen" value="0.23" />
-  <xacro:property name="basewidth" value="0.26" />
-  <xacro:property name="basethick" value="0.01" />
-  <xacro:property name="wheeldiam" value="0.065" />
-  <xacro:property name="wheelwidth" value="0.0325" />
+  <xacro:property name="package_name" value="hello_robot" />
+  <xacro:property name="robot_name" value="hello_robot" />
+  <xacro:include filename="$(find ${package_name})/urdf/hello_robot.gazebo.xacro" />
+  <xacro:include filename="$(find ${package_name})/urdf/include/common_macros.urdf.xacro" />
+  <xacro:property name="baselen" value="0.24" />
+  <xacro:property name="basewidth" value="0.15" />
+  <xacro:property name="basethick" value="0.003" />
+  <xacro:property name="wheeldiam" value="0.056" />
+  <xacro:property name="wheelwidth" value="0.037" />
   <xacro:property name="pi" value="3.1415" />
-  <material name="white">
-    <color rgba="1 1 1 1"/>
-  </material>
-  <material name="black">
-    <color rgba=".05 .05 .05 1"/>
-  </material>
-  <!-- ======================= Intertial macros ===============================-->
-  <!-- ===================== Cylinder intertia xacro =============================
-  Xacro with the intertial block of a cylinder. For more detail information and usage, see:
-    https://github.com/pxalcantara/mobile_robot_description/wiki/Inertia-xacro
-  params:
-  - m [float]: link mass;
-  - r [float]: cylinder radius;
-  - l [float]: cylinder lenght (height);
-  -->
-  <xacro:macro name="wheel_inertia" params="m r l o_xyz:='0.0 0.0 0.0' o_rpy:='0.0 0.0 0.0'">
-    <inertial>
-      <mass value="${m}"/>
-      <inertia ixx="${m*(3*r*r+l*l)/12}" ixy = "0" ixz = "0"
-               iyy="${m*(3*r*r+l*l)/12}" iyz = "0" izz="${m*r*r/2}"/>
-      <origin xyz="${o_xyz}" rpy="${o_rpy}" />
-    </inertial>
-  </xacro:macro>
-  <!-- ===================== Box intertia xacro ==================================
-  Xacro with the intertial block of a box. For more detail information and usage, see:
-    https://github.com/pxalcantara/mobile_robot_description/wiki/Inertia-xacro
-  params:
-  - m [float]: link mass;
-  - x [float]: link dimension on the X-axis;
-  - y [float]: link dimension on the Y-axis;
-  - z [float]: link dimension on the Z-axis;
--->
-<xacro:macro name="base_inertia" params="m x y z o_xyz:='0.0 0.0 0.0' o_rpy:='0.0 0.0 0.0'">
-    <inertial>
-      <mass value="${m}"/>
-      <inertia ixx="${m / 12.0 * (y*y + z*z)}" ixy="0.0" ixz="0.0"
-               iyy="${m / 12.0 * (x*x + z*z)}" iyz="0.0"
-               izz="${m / 12.0 * (x*x + y*y)}"/>
-      <origin xyz="${o_xyz}" rpy="${o_rpy}" />
-    </inertial>
-  </xacro:macro>
   <link name="base_link">
     <visual>
@@ -60,64 +23,19 @@
       </geometry>
     </collision>
-    <xacro:base_inertia m="1"
+    <xacro:base_inertia m="1.065"
     x="${baselen}" y="${basewidth}" z="${basethick}"
     o_xyz="0.0 0.0 0.0" o_rpy="0.0 0.0 0.0"
     />
   </link>
-  <xacro:macro name="wheel" params="prefix suffix reflectfrontback reflectside">
-    <link name="${prefix}_${suffix}_wheel">
-      <visual>
-        <origin xyz="0 0 0" rpy="${pi/2} 0 0" />
-        <geometry>
-          <cylinder radius="${wheeldiam/2}" length="${wheelwidth}"/>
-        </geometry>
-        <material name="black"/>
-      </visual>
-      <collision>
-        <origin xyz="0 0 0" rpy="${pi/2} 0 0" />
-        <geometry>
-          <cylinder radius="${wheeldiam/2}" length="${wheelwidth}"/>
-        </geometry>
-      </collision>
-      <xacro:wheel_inertia m="0.1" r="${wheeldiam/2}" l="${wheelwidth}"
-      o_xyz="0.0 0.0 0.0" o_rpy="0.0 0.0 0.0"
-      />
-    </link>
-    <joint name="${prefix}_${suffix}_wheel_joint" type="continuous">
-      <axis xyz="0 1 0" rpy="0 0 0" />
-      <parent link="base_link"/>
-      <child link="${prefix}_${suffix}_wheel"/>
-      <origin xyz="${baselen*reflectfrontback/3} ${((basewidth/2)+wheelwidth/2)*reflectside} ${-wheeldiam/2}" rpy="0 0 0"/>
-    </joint>
-        <!-- This block provides the simulator (Gazebo) with information on a few additional
-    physical properties. See http://gazebosim.org/tutorials/?tut=ros_urdf for more-->
-    <gazebo reference="${prefix}_${suffix}_wheel">
-      <mu1 value="200.0"/>
-      <mu2 value="100.0"/>
-      <kp value="10000000.0" />
-      <kd value="1.0" />
-      <material>Gazebo/Grey</material>
-    </gazebo>
-    <!-- This block connects the wheel joint to an actuator (motor), which informs both
-    simulation and visualization of the robot -->
-    <transmission name="${prefix}_${suffix}_wheel_trans">
-      <type>transmission_interface/SimpleTransmission</type>
-      <actuator name="${prefix}_${suffix}_wheel_motor">
-        <mechanicalReduction>1</mechanicalReduction>
-      </actuator>
-      <joint name="${prefix}_${suffix}_wheel_joint">
-        <hardwareInterface>VelocityJointInterface</hardwareInterface>
-      </joint>
-    </transmission>
-  </xacro:macro>
-  <xacro:wheel prefix="left" suffix="front" reflectfrontback="1" reflectside="1"/>
-  <xacro:wheel prefix="left" suffix="back" reflectfrontback="-1" reflectside="1"/>
-  <xacro:wheel prefix="right" suffix="front" reflectfrontback="1" reflectside="-1"/>
-  <xacro:wheel prefix="right" suffix="back" reflectfrontback="-1" reflectside="-1"/>
-  <!-- Gazebo plugin for ROS Control -->
-  <gazebo>
-    <plugin name="gazebo_ros_control" filename="libgazebo_ros_control.so">
-      <robotNamespace>/</robotNamespace>
-    </plugin>
-  </gazebo>
+  <link name="base_footprint" />
+  <!-- Joint to connect base_footprint with base_link -->
+  <joint name="base_footprint_joint" type="fixed">
+    <parent link="base_footprint"/>
+    <child link="base_link" />
+    <origin xyz="0 0 ${-wheeldiam}" rpy="0 0 0" />
+  </joint>
+  <xacro:wheel prefix="left" suffix="front" reflectfrontback="1" reflectside="1" m="0.087" r="${wheeldiam/2}" l="${wheelwidth}" />
+  <xacro:wheel prefix="left" suffix="back" reflectfrontback="-1" reflectside="1" m="0.087" r="${wheeldiam/2}" l="${wheelwidth}" />
+  <xacro:wheel prefix="right" suffix="front" reflectfrontback="1" reflectside="-1" m="0.087" r="${wheeldiam/2}" l="${wheelwidth}" />
+  <xacro:wheel prefix="right" suffix="back" reflectfrontback="-1" reflectside="-1" m="0.087" r="${wheeldiam/2}" l="${wheelwidth}" />
 </robot>

Commit message: added base_footprint

File: urdf/hello_robot.xacro (robot description, xacro)
@@ -11,4 +11,11 @@
   <xacro:property name="wheelwidth" value="0.037" />
   <xacro:property name="pi" value="3.1415" />
+  <link name="base_footprint" />
+  <!-- Joint to connect base_footprint with base_link -->
+  <joint name="base_footprint_joint" type="fixed">
+    <parent link="base_footprint"/>
+    <child link="base_link" />
+    <origin xyz="0 0 ${-wheeldiam}" rpy="0 0 0" />
+  </joint>
   <link name="base_link">
     <visual>
@@ -28,11 +35,4 @@
     />
   </link>
-  <link name="base_footprint" />
-  <!-- Joint to connect base_footprint with base_link -->
-  <joint name="base_footprint_joint" type="fixed">
-    <parent link="base_footprint"/>
-    <child link="base_link" />
-    <origin xyz="0 0 ${-wheeldiam}" rpy="0 0 0" />
-  </joint>
   <xacro:wheel prefix="left" suffix="front" reflectfrontback="1" reflectside="1" m="0.087" r="${wheeldiam/2}" l="${wheelwidth}" />
   <xacro:wheel prefix="left" suffix="back" reflectfrontback="-1" reflectside="1" m="0.087" r="${wheeldiam/2}" l="${wheelwidth}" />
