Commit message: Added laser scanner

File: urdf/hello_robot.urdf.xacro (robot description, xacro)
@@ -5,4 +5,7 @@
   <xacro:include filename="$(find ${package_name})/urdf/hello_robot.gazebo.xacro" />
   <xacro:include filename="$(find ${package_name})/urdf/include/common_macros.urdf.xacro" />
+  <xacro:include filename="$(find ${package_name})/urdf/include/common_sensors.xacro" />
+  <xacro:property name="sensor_yaml" value="$(find ${package_name})/config/sensors.yaml" />
+  <xacro:property name="sensor_prop" value="${load_yaml(sensor_yaml)}"/>
   <xacro:property name="baselen" value="0.24" />
   <xacro:property name="basewidth" value="0.15" />
@@ -39,3 +42,7 @@
   <xacro:wheel prefix="right" suffix="front" reflectfrontback="1" reflectside="-1" m="0.087" r="${wheeldiam/2}" l="${wheelwidth}" />
   <xacro:wheel prefix="right" suffix="back" reflectfrontback="-1" reflectside="-1" m="0.087" r="${wheeldiam/2}" l="${wheelwidth}" />
+  <!-- Sensors -->
+  <xacro:gpu_laser prefix="rplidar" parent_link="base_link"
+                   sensor_prop="${sensor_prop}">
+  </xacro:gpu_laser>
 </robot>

File: urdf/include/common_macros.urdf.xacro (robot description, xacro)
@@ -28,5 +28,5 @@
             </geometry>
         </collision>
-        <xacro:wheel_inertia m="${m}" r="${r}" l="${l}"
+        <xacro:cylinder_inertia m="${m}" r="${r}" l="${l}"
         o_xyz="0.0 0.0 0.0" o_rpy="0.0 0.0 0.0"
         />
@@ -68,5 +68,5 @@
   - l [float]: cylinder lenght (height);
   -->
-  <xacro:macro name="wheel_inertia" params="m r l o_xyz:='0.0 0.0 0.0' o_rpy:='0.0 0.0 0.0'">
+  <xacro:macro name="cylinder_inertia" params="m r l o_xyz:='0.0 0.0 0.0' o_rpy:='0.0 0.0 0.0'">
     <inertial>
       <mass value="${m}"/>

Commit message: Working on parameters

File: urdf/hello_robot.urdf.xacro (robot description, xacro)
@@ -13,5 +13,8 @@
   <xacro:property name="wheeldiam" value="0.056" />
   <xacro:property name="wheelwidth" value="0.037" />
-  <xacro:property name="pi" value="3.1415" />
+  <xacro:property name="wheel_x_pos" value="0.10" />
+  <xacro:property name="wheel_y_pos" value="${basewidth/2+.035}" />
+  <xacro:property name="wheel_z_pos" value="${-((basethick/2)+(wheeldiam/2)+.01)}" />
+  <xacro:property name="pi" value="3.1415926535" />
   <link name="base_footprint" />
   <!-- Joint to connect base_footprint with base_link -->
@@ -19,5 +22,5 @@
     <parent link="base_footprint"/>
     <child link="base_link" />
-    <origin xyz="0 0 ${-wheeldiam}" rpy="0 0 0" />
+    <origin xyz="0 0 ${(wheeldiam/2)+(-wheel_z_pos)}" rpy="0 0 0" />
   </joint>
   <link name="base_link">
@@ -38,8 +41,8 @@
     />
   </link>
-  <xacro:wheel prefix="left" suffix="front" reflectfrontback="1" reflectside="1" m="0.087" r="${wheeldiam/2}" l="${wheelwidth}" />
-  <xacro:wheel prefix="left" suffix="back" reflectfrontback="-1" reflectside="1" m="0.087" r="${wheeldiam/2}" l="${wheelwidth}" />
-  <xacro:wheel prefix="right" suffix="front" reflectfrontback="1" reflectside="-1" m="0.087" r="${wheeldiam/2}" l="${wheelwidth}" />
-  <xacro:wheel prefix="right" suffix="back" reflectfrontback="-1" reflectside="-1" m="0.087" r="${wheeldiam/2}" l="${wheelwidth}" />
+  <xacro:wheel prefix="left" suffix="front" m="0.087" r="${wheeldiam/2}" l="${wheelwidth}" x_pos="${wheel_x_pos}" y_pos="${wheel_y_pos}" z_pos="${wheel_z_pos}"/>
+  <xacro:wheel prefix="left" suffix="back" m="0.087" r="${wheeldiam/2}" l="${wheelwidth}" x_pos="${-wheel_x_pos}" y_pos="${wheel_y_pos}" z_pos="${wheel_z_pos}"/>
+  <xacro:wheel prefix="right" suffix="front" m="0.087" r="${wheeldiam/2}" l="${wheelwidth}" x_pos="${wheel_x_pos}" y_pos="${-wheel_y_pos}" z_pos="${wheel_z_pos}"/>
+  <xacro:wheel prefix="right" suffix="back" m="0.087" r="${wheeldiam/2}" l="${wheelwidth}" x_pos="${-wheel_x_pos}" y_pos="${-wheel_y_pos}" z_pos="${wheel_z_pos}"/>
   <!-- Sensors -->
   <xacro:gpu_laser prefix="rplidar" parent_link="base_link"

File: urdf/include/common_macros.urdf.xacro (robot description, xacro)
@@ -10,35 +10,37 @@
   - prefix [string]: left or right
   - suffix [string]: front or back
-  - reflectfrontback [int]: 1(front) or -1(back)
   - reflectside [int]: 1(left) or -1(right)
+  - x_pos [float]: moves wheel forward or backward from the origin of the base
+  - y_pos [float]: moves wheel left or right from the origin of the base
+  - z_pos [float]: moves wheel up or down from the origin of the base
   -->
-    <xacro:macro name="wheel" params="prefix suffix reflectfrontback reflectside m r l">
-        <link name="${prefix}_${suffix}_wheel">
-        <visual>
-            <origin xyz="0 0 0" rpy="${pi/2} 0 0" />
-            <geometry>
-            <cylinder radius="${r}" length="${l}"/>
-            </geometry>
-            <material name="black"/>
-        </visual>
-        <collision>
-            <origin xyz="0 0 0" rpy="${pi/2} 0 0" />
-            <geometry>
-            <cylinder radius="${r}" length="${l}"/>
-            </geometry>
-        </collision>
-        <xacro:cylinder_inertia m="${m}" r="${r}" l="${l}"
+  <xacro:macro name="wheel" params="prefix suffix m r l x_pos y_pos z_pos">
+    <link name="${prefix}_${suffix}_wheel">
+      <visual>
+          <origin xyz="0 0 0" rpy="${pi/2} 0 0" />
+          <geometry>
+          <cylinder radius="${r}" length="${l}"/>
+          </geometry>
+          <material name="black"/>
+      </visual>
+      <collision>
+          <origin xyz="0 0 0" rpy="${pi/2} 0 0" />
+          <geometry>
+          <cylinder radius="${r}" length="${l}"/>
+          </geometry>
+      </collision>
+      <xacro:cylinder_inertia m="${m}" r="${r}" l="${l}"
         o_xyz="0.0 0.0 0.0" o_rpy="0.0 0.0 0.0"
-        />
-        </link>
-        <joint name="${prefix}_${suffix}_wheel_joint" type="continuous">
+      />
+    </link>
+      <joint name="${prefix}_${suffix}_wheel_joint" type="continuous">
         <axis xyz="0 1 0" rpy="0 0 0" />
         <parent link="base_link"/>
         <child link="${prefix}_${suffix}_wheel"/>
-        <origin xyz="${baselen*reflectfrontback/3} ${((basewidth/2)+l/2)*reflectside} ${-r}" rpy="0 0 0"/>
-        </joint>
-            <!-- This block provides the simulator (Gazebo) with information on a few additional
-        physical properties. See http://gazebosim.org/tutorials/?tut=ros_urdf for more-->
-        <gazebo reference="${prefix}_${suffix}_wheel">
+        <origin xyz="${x_pos} ${y_pos} ${z_pos}" rpy="0 0 0"/>
+      </joint>
+          <!-- This block provides the simulator (Gazebo) with information on a few additional
+      physical properties. See http://gazebosim.org/tutorials/?tut=ros_urdf for more-->
+      <gazebo reference="${prefix}_${suffix}_wheel">
         <mu1 value="200.0"/>
         <mu2 value="100.0"/>
@@ -46,17 +48,17 @@
         <kd value="1.0" />
         <material>Gazebo/Grey</material>
-        </gazebo>
-        <!-- This block connects the wheel joint to an actuator (motor), which informs both
-        simulation and visualization of the robot -->
-        <transmission name="${prefix}_${suffix}_wheel_trans">
-        <type>transmission_interface/SimpleTransmission</type>
-        <actuator name="${prefix}_${suffix}_wheel_motor">
-            <mechanicalReduction>1</mechanicalReduction>
-        </actuator>
-        <joint name="${prefix}_${suffix}_wheel_joint">
-            <hardwareInterface>VelocityJointInterface</hardwareInterface>
-        </joint>
-        </transmission>
-    </xacro:macro>
+      </gazebo>
+      <!-- This block connects the wheel joint to an actuator (motor), which informs both
+      simulation and visualization of the robot -->
+    <transmission name="${prefix}_${suffix}_wheel_trans">
+      <type>transmission_interface/SimpleTransmission</type>
+      <actuator name="${prefix}_${suffix}_wheel_motor">
+          <mechanicalReduction>1</mechanicalReduction>
+      </actuator>
+      <joint name="${prefix}_${suffix}_wheel_joint">
+          <hardwareInterface>VelocityJointInterface</hardwareInterface>
+      </joint>
+    </transmission>
+  </xacro:macro>
   <!-- ======================= Intertial macros ===============================-->
   <!-- ===================== Cylinder intertia xacro =============================

Commit message: Dimensional updates to hello_robot xacro

File: urdf/hello_robot.urdf.xacro (robot description, xacro)
@@ -8,12 +8,12 @@
   <xacro:property name="sensor_yaml" value="$(find ${package_name})/config/sensors.yaml" />
   <xacro:property name="sensor_prop" value="${load_yaml(sensor_yaml)}"/>
-  <xacro:property name="baselen" value="0.24" />
-  <xacro:property name="basewidth" value="0.15" />
+  <xacro:property name="baselen" value="0.260" />
+  <xacro:property name="basewidth" value="0.152" />
   <xacro:property name="basethick" value="0.003" />
   <xacro:property name="wheeldiam" value="0.056" />
-  <xacro:property name="wheelwidth" value="0.037" />
+  <xacro:property name="wheelwidth" value="0.038" />
   <xacro:property name="wheel_x_pos" value="0.10" />
-  <xacro:property name="wheel_y_pos" value="${basewidth/2+.035}" />
-  <xacro:property name="wheel_z_pos" value="${-((basethick/2)+(wheeldiam/2)+.01)}" />
+  <xacro:property name="wheel_y_pos" value="${wheelwidth/2+basewidth/2+.013}" />
+  <xacro:property name="wheel_z_pos" value="${-((basethick/2)+(wheeldiam/2)+.007)}" />
   <xacro:property name="pi" value="3.1415926535" />
   <link name="base_footprint" />

Commit message: Laser sensor position update

File: urdf/hello_robot.urdf.xacro (robot description, xacro)
@@ -13,5 +13,5 @@
   <xacro:property name="wheeldiam" value="0.056" />
   <xacro:property name="wheelwidth" value="0.038" />
-  <xacro:property name="wheel_x_pos" value="0.10" />
+  <xacro:property name="wheel_x_pos" value="${baselen/2}" />
   <xacro:property name="wheel_y_pos" value="${wheelwidth/2+basewidth/2+.013}" />
   <xacro:property name="wheel_z_pos" value="${-((basethick/2)+(wheeldiam/2)+.007)}" />
@@ -41,8 +41,8 @@
     />
   </link>
-  <xacro:wheel prefix="left" suffix="front" m="0.087" r="${wheeldiam/2}" l="${wheelwidth}" x_pos="${wheel_x_pos}" y_pos="${wheel_y_pos}" z_pos="${wheel_z_pos}"/>
-  <xacro:wheel prefix="left" suffix="back" m="0.087" r="${wheeldiam/2}" l="${wheelwidth}" x_pos="${-wheel_x_pos}" y_pos="${wheel_y_pos}" z_pos="${wheel_z_pos}"/>
-  <xacro:wheel prefix="right" suffix="front" m="0.087" r="${wheeldiam/2}" l="${wheelwidth}" x_pos="${wheel_x_pos}" y_pos="${-wheel_y_pos}" z_pos="${wheel_z_pos}"/>
-  <xacro:wheel prefix="right" suffix="back" m="0.087" r="${wheeldiam/2}" l="${wheelwidth}" x_pos="${-wheel_x_pos}" y_pos="${-wheel_y_pos}" z_pos="${wheel_z_pos}"/>
+  <xacro:wheel prefix="left" suffix="front" m="0.087" r="${wheeldiam/2}" l="${wheelwidth}" x_pos="${wheel_x_pos-.057}" y_pos="${wheel_y_pos}" z_pos="${wheel_z_pos}"/>
+  <xacro:wheel prefix="left" suffix="back" m="0.087" r="${wheeldiam/2}" l="${wheelwidth}" x_pos="${-wheel_x_pos+.042}" y_pos="${wheel_y_pos}" z_pos="${wheel_z_pos}"/>
+  <xacro:wheel prefix="right" suffix="front" m="0.087" r="${wheeldiam/2}" l="${wheelwidth}" x_pos="${wheel_x_pos-.057}" y_pos="${-wheel_y_pos}" z_pos="${wheel_z_pos}"/>
+  <xacro:wheel prefix="right" suffix="back" m="0.087" r="${wheeldiam/2}" l="${wheelwidth}" x_pos="${-wheel_x_pos+.042}" y_pos="${-wheel_y_pos}" z_pos="${wheel_z_pos}"/>
   <!-- Sensors -->
   <xacro:gpu_laser prefix="rplidar" parent_link="base_link"
