Commit message: reorganized hello_robot again into packages

File: hello_robot_description/urdf/hello_robot.urdf.xacro (robot description, xacro)
@@ -1,9 +1,9 @@
 <?xml version="1.0"?>
 <robot name="hello_robot" xmlns:xacro="http://www.ros.org/wiki/xacro">
-  <xacro:property name="package_name" value="hello_robot" />
+  <xacro:property name="package_name" value="hello_robot_description" />
   <xacro:property name="robot_name" value="hello_robot" />
-  <xacro:include filename="$(find ${package_name})/description/hello_robot.gazebo.xacro" />
-  <xacro:include filename="$(find ${package_name})/description/include/common_macros.urdf.xacro" />
-  <xacro:include filename="$(find ${package_name})/description/include/common_sensors.xacro" />
+  <xacro:include filename="$(find ${package_name})/urdf/hello_robot.gazebo.xacro" />
+  <xacro:include filename="$(find ${package_name})/urdf/include/common_macros.urdf.xacro" />
+  <xacro:include filename="$(find ${package_name})/urdf/include/common_sensors.xacro" />
   <xacro:property name="sensor_yaml" value="$(find ${package_name})/config/sensors.yaml" />
   <xacro:property name="sensor_prop" value="${load_yaml(sensor_yaml)}"/>

Commit message: tuning navigation stack

File: hello_robot_description/urdf/hello_robot.urdf.xacro (robot description, xacro)
@@ -17,4 +17,5 @@
   <xacro:property name="wheel_z_pos" value="${-((basethick/2)+(wheeldiam/2)+.007)}" />
   <xacro:property name="pi" value="3.1415926535" />
+  <xacro:property name="collision_inflation" value="1.1" />
   <link name="base_footprint" />
   <!-- Joint to connect base_footprint with base_link -->
@@ -33,5 +34,5 @@
     <collision>
       <geometry>
-        <box size="${baselen} ${basewidth} ${basethick}" />
+        <box size="${baselen*collision_inflation} ${basewidth*collision_inflation} ${basethick*collision_inflation}" />
       </geometry>
     </collision>
@@ -41,8 +42,8 @@
     />
   </link>
-  <xacro:wheel prefix="left" suffix="front" m="0.087" r="${wheeldiam/2}" l="${wheelwidth}" x_pos="${wheel_x_pos-.057}" y_pos="${wheel_y_pos}" z_pos="${wheel_z_pos}"/>
-  <xacro:wheel prefix="left" suffix="back" m="0.087" r="${wheeldiam/2}" l="${wheelwidth}" x_pos="${-wheel_x_pos+.042}" y_pos="${wheel_y_pos}" z_pos="${wheel_z_pos}"/>
-  <xacro:wheel prefix="right" suffix="front" m="0.087" r="${wheeldiam/2}" l="${wheelwidth}" x_pos="${wheel_x_pos-.057}" y_pos="${-wheel_y_pos}" z_pos="${wheel_z_pos}"/>
-  <xacro:wheel prefix="right" suffix="back" m="0.087" r="${wheeldiam/2}" l="${wheelwidth}" x_pos="${-wheel_x_pos+.042}" y_pos="${-wheel_y_pos}" z_pos="${wheel_z_pos}"/>
+  <xacro:wheel prefix="left" suffix="front" m="0.087" r="${wheeldiam/2}" l="${wheelwidth}" x_pos="${wheel_x_pos-.057}" y_pos="${wheel_y_pos}" z_pos="${wheel_z_pos}" collision_inflation="${collision_inflation}"/>
+  <xacro:wheel prefix="left" suffix="back" m="0.087" r="${wheeldiam/2}" l="${wheelwidth}" x_pos="${-wheel_x_pos+.042}" y_pos="${wheel_y_pos}" z_pos="${wheel_z_pos}" collision_inflation="${collision_inflation}"/>
+  <xacro:wheel prefix="right" suffix="front" m="0.087" r="${wheeldiam/2}" l="${wheelwidth}" x_pos="${wheel_x_pos-.057}" y_pos="${-wheel_y_pos}" z_pos="${wheel_z_pos}" collision_inflation="${collision_inflation}"/>
+  <xacro:wheel prefix="right" suffix="back" m="0.087" r="${wheeldiam/2}" l="${wheelwidth}" x_pos="${-wheel_x_pos+.042}" y_pos="${-wheel_y_pos}" z_pos="${wheel_z_pos}" collision_inflation="${collision_inflation}"/>
   <!-- Sensors -->
   <xacro:gpu_laser prefix="rplidar" parent_link="base_link"

File: hello_robot_description/urdf/include/common_macros.urdf.xacro (robot description, xacro)
@@ -15,5 +15,5 @@
   - z_pos [float]: moves wheel up or down from the origin of the base
   -->
-  <xacro:macro name="wheel" params="prefix suffix m r l x_pos y_pos z_pos">
+  <xacro:macro name="wheel" params="prefix suffix m r l x_pos y_pos z_pos collision_inflation">
     <link name="${prefix}_${suffix}_wheel">
       <visual>
@@ -27,9 +27,9 @@
           <origin xyz="0 0 0" rpy="${pi/2} 0 0" />
           <geometry>
-          <cylinder radius="${r}" length="${l}"/>
+          <cylinder radius="${r*collision_inflation}" length="${l*collision_inflation}"/>
           </geometry>
       </collision>
       <xacro:cylinder_inertia m="${m}" r="${r}" l="${l}"
-        o_xyz="0.0 0.0 0.0" o_rpy="0.0 0.0 0.0"
+        o_xyz="0.0 0.0 0.0" o_rpy="${pi/2} 0.0 0.0"
       />
     </link>
@@ -44,7 +44,8 @@
       <gazebo reference="${prefix}_${suffix}_wheel">
         <mu1 value="200.0"/>
-        <mu2 value="100.0"/>
+        <mu2 value="200.0"/>
         <kp value="10000000.0" />
         <kd value="1.0" />
+        <minDepth>0.08</minDepth>
         <material>Gazebo/Grey</material>
       </gazebo>
